File: eagle/hsArduino.brd (EAGLE design)
At the start: 86 x 66 mm, 119 parts, among them IC1 R-78B5.0-1.5, IC2 REG1117, IC3 LMV321M5, IC4 74LVC1G14DBV, IC5 74LVC1G14DBV, IC6 MAX3232CSE, Q1 IRLML6401, Q2 IRLML6401, Q3 25MHz, Q4 16MHz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

Commit message: BOM
Parts:
- removed D3: (no value), diode:SOT54H
- added R37: CG0603-05, varistor:CT/CN0603
- R1: value 680k -> 1M
- R22, R34: value 22k -> 15k
Connections:
- net GND: now also R37.2; no longer D3.A
- net N$38: now also R37.1; no longer D3.C
Routing:
- net N$38: track 25.9 -> 26.5 mm, vias 1 -> 0
- net GND: track 114.7 -> 114.5 mm, vias 28 -> 29
Changed lines of the file:
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@@
 <attribute name="VALUE" x="11.43" y="62.992" size="1.016" layer="27" ratio="10" rot="R270"/>
 </element>
-<element name="R1" library="rcl" package="R0805" value="680k" x="13.335" y="53.0225" smashed="yes">
+<element name="R1" library="rcl" package="R0805" value="1M" x="13.335" y="53.0225" smashed="yes">
 <attribute name="NAME" x="14.9225" y="53.0225" size="1.016" layer="25"/>
 <attribute name="VALUE" x="14.9225" y="51.7525" size="1.016" layer="27"/>
@@
 <attribute name="VALUE" x="74.295" y="20.0025" size="1.016" layer="27"/>
 </element>
-<element name="R22" library="rcl" package="R0805" value="22k" x="60.96" y="21.59" smashed="yes" rot="R180">
+<element name="R22" library="rcl" package="R0805" value="15k" x="60.96" y="21.59" smashed="yes" rot="R180">
 <attribute name="NAME" x="57.15" y="20.955" size="1.016" layer="25"/>
 <attribute name="VALUE" x="59.69" y="22.225" size="1.016" layer="27"/>
 </element>
-<element name="R34" library="rcl" package="R0805" value="22k" x="60.96" y="19.05" smashed="yes" rot="R180">
+<element name="R34" library="rcl" package="R0805" value="15k" x="60.96" y="19.05" smashed="yes" rot="R180">
 <attribute name="NAME" x="57.15" y="18.415" size="1.016" layer="25"/>
 <attribute name="VALUE" x="59.69" y="19.685" size="1.016" layer="27"/>
@@
 <attribute name="NAME" x="1.482" y="34.29" size="1.016" layer="25" ratio="10" rot="R270"/>
 <attribute name="VALUE" x="-1.185" y="34.29" size="1.27" layer="27" ratio="10" rot="R270"/>
-</element>
-<element name="D3" library="diode" package="SOT54H" value="" x="71.755" y="43.18" smashed="yes" rot="R90">
-<attribute name="NAME" x="71.755" y="44.45" size="1.016" layer="25" ratio="10" rot="R180"/>
-<attribute name="VALUE" x="73.025" y="46.355" size="1.27" layer="27" ratio="10" rot="R90"/>
 </element>
 <element name="C16" library="rcl" package="C0805K" value="4n7" x="13.335" y="20.955" smashed="yes" rot="R180">
@@
 <element name="R8" library="varistor" package="CT/CN0603" value="CG0603-05" x="73.025" y="48.26" smashed="yes" rot="R270">
 <attribute name="NAME" x="73.6125" y="49.6175" size="1.016" layer="25" rot="R90"/>
-<attribute name="VALUE" x="75.025" y="43.585" size="1.016" layer="27" rot="R90"/>
+<attribute name="VALUE" x="75.025" y="41.68" size="1.016" layer="27" rot="R90"/>
 </element>
 <element name="IC3" library="linear" package="SOT23-5" value="LMV321M5" x="59.055" y="52.705" smashed="yes">
@@
 <attribute name="VALUE" x="55.885" y="51.07" size="1.016" layer="28" rot="MR90"/>
 </element>
+<element name="R37" library="varistor" package="CT/CN0603" value="CG0603-05" x="73.025" y="43.18" rot="R90"/>
 </elements>
 <signals>
@@
 <contactref element="X1" pad="2"/>
 <contactref element="X4" pad="2"/>
-<contactref element="D3" pad="A"/>
 <contactref element="SV3" pad="4"/>
 <contactref element="SV3" pad="5"/>
@@
 <wire x1="64.77" y1="47.3075" x2="65.3575" y2="47.3075" width="0.4064" layer="1"/>
 <wire x1="65.3575" y1="47.3075" x2="65.405" y2="47.26" width="0.4064" layer="1"/>
-<wire x1="73.025" y1="47.26" x2="73.025" y2="45.72" width="0.4064" layer="1"/>
-<wire x1="73.025" y1="45.72" x2="71.755" y2="44.45" width="0.4064" layer="1"/>
 <wire x1="50.165" y1="53.655" x2="50.165" y2="53.975" width="0.4064" layer="1"/>
 <wire x1="50.165" y1="53.975" x2="51.435" y2="55.245" width="0.4064" layer="1"/>
@@
 <wire x1="16.8275" y1="27.6225" x2="16.51" y2="27.94" width="0.4064" layer="1"/>
 <via x="16.51" y="27.94" extent="1-16" drill="0.6"/>
+<contactref element="R37" pad="2"/>
+<wire x1="73.025" y1="47.26" x2="73.025" y2="45.72" width="0.4064" layer="1"/>
+<wire x1="73.025" y1="45.72" x2="73.025" y2="44.18" width="0.4064" layer="1"/>
+<via x="73.025" y="45.72" extent="1-16" drill="0.6"/>
 </signal>
 <signal name="N$1">
@@
 <contactref element="X3" pad="1"/>
 <contactref element="R13" pad="1"/>
-<contactref element="D3" pad="C"/>
 <wire x1="80.835" y1="55.88" x2="79.375" y2="55.88" width="0.4064" layer="1"/>
 <wire x1="79.375" y1="55.88" x2="74.93" y2="51.435" width="0.4064" layer="1"/>
-<wire x1="74.93" y1="51.435" x2="74.93" y2="45.085" width="0.4064" layer="1"/>
-<wire x1="74.93" y1="45.085" x2="71.755" y2="41.91" width="0.4064" layer="1"/>
-<wire x1="71.755" y1="41.91" x2="71.755" y2="40.64" width="0.4064" layer="16"/>
-<wire x1="71.755" y1="40.64" x2="68.58" y2="37.465" width="0.4064" layer="16"/>
-<via x="68.58" y="37.465" extent="1-16" drill="0.6"/>
 <wire x1="68.58" y1="37.465" x2="66.99" y2="37.465" width="0.4064" layer="1"/>
+<contactref element="R37" pad="1"/>
+<wire x1="74.93" y1="51.435" x2="74.93" y2="43.18" width="0.4064" layer="1"/>
+<wire x1="74.93" y1="43.18" x2="73.9775" y2="42.2275" width="0.4064" layer="1"/>
+<wire x1="73.9775" y1="42.2275" x2="73.0725" y2="42.2275" width="0.4064" layer="1"/>
+<wire x1="73.0725" y1="42.2275" x2="73.025" y2="42.18" width="0.4064" layer="1"/>
+<wire x1="73.025" y1="42.18" x2="73.025" y2="41.91" width="0.4064" layer="1"/>
+<wire x1="73.025" y1="41.91" x2="68.58" y2="37.465" width="0.4064" layer="1"/>
 </signal>
 <signal name="PD7">
