File: eagle/hsArduino.sch (EAGLE design)
At the start: 119 parts, among them IC1 R-78B5.0-1.5, IC2 REG1117, IC3 LMV321M5, IC4 74LVC1G14DBV, IC5 74LVC1G14DBV, IC6 MAX3232CSE, Q1 IRLML6401, Q2 IRLML6401, Q3 25MHz, Q4 16MHz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

Commit message: BOM
Parts:
- removed D3: (no value), diode:DIODE-SOT54H
- added R37: CG0603-05, varistor:VARISTORCN0603
- R1: value 680k -> 1M
- R22, R34: value 22k -> 15k
Connections:
- net GND: now also R37.2; no longer D3.A
- net N$38: now also R37.1; no longer D3.C
Other:
- moved on the sheet: D4, X3-1, X3-2
Changed lines of the file:
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@@
 <part name="GND27" library="supply1" deviceset="GND" device=""/>
 <part name="C1" library="rcl" deviceset="CPOL-EU" device="E2.5-7" value="100µ"/>
-<part name="R1" library="rcl" deviceset="R-EU_" device="R0805" value="680k"/>
+<part name="R1" library="rcl" deviceset="R-EU_" device="R0805" value="1M"/>
 <part name="GND28" library="supply1" deviceset="GND" device=""/>
 <part name="GND29" library="supply1" deviceset="GND" device=""/>
@@
 <part name="R26" library="rcl" deviceset="R-EU_" device="R0805" value="220"/>
 <part name="R27" library="rcl" deviceset="R-EU_" device="R0805" value="220"/>
-<part name="R22" library="rcl" deviceset="R-EU_" device="R0805" value="22k"/>
-<part name="R34" library="rcl" deviceset="R-EU_" device="R0805" value="22k"/>
+<part name="R22" library="rcl" deviceset="R-EU_" device="R0805" value="15k"/>
+<part name="R34" library="rcl" deviceset="R-EU_" device="R0805" value="15k"/>
 <part name="P+13" library="supply1" deviceset="+5V" device=""/>
 <part name="D4" library="diode" deviceset="BAS40-04" device=""/>
@@
 <part name="X6" library="con-wago-508" deviceset="W237-02P" device=""/>
 <part name="X8" library="con-wago-508" deviceset="W237-02P" device=""/>
-<part name="D3" library="diode" deviceset="DIODE-" device="SOT54H"/>
 <part name="P+10" library="supply1" deviceset="+5V" device=""/>
 <part name="GND36" library="supply1" deviceset="GND" device=""/>
@@
 <part name="C115" library="rcl" deviceset="C-EU" device="C0805K" value="100n"/>
 <part name="GND52" library="supply1" deviceset="GND" device=""/>
+<part name="R37" library="varistor" deviceset="VARISTOR" device="CN0603" value="CG0603-05"/>
 </parts>
 <sheets>
@@
 </instance>
 <instance part="P+13" gate="1" x="228.6" y="66.04"/>
-<instance part="D4" gate="G$1" x="210.82" y="104.14" rot="MR90"/>
-<instance part="X3" gate="-1" x="220.98" y="88.9" rot="R90"/>
-<instance part="X3" gate="-2" x="210.82" y="88.9" rot="R90"/>
+<instance part="D4" gate="G$1" x="205.74" y="104.14" rot="MR90"/>
+<instance part="X3" gate="-1" x="220.98" y="86.36" rot="R90"/>
+<instance part="X3" gate="-2" x="205.74" y="86.36" rot="R90"/>
 <instance part="R13" gate="G$1" x="220.98" y="99.06" rot="R90"/>
 <instance part="R12" gate="G$1" x="220.98" y="109.22" rot="R90"/>
 <instance part="P+14" gate="1" x="220.98" y="121.92"/>
-<instance part="GND34" gate="1" x="208.28" y="96.52" rot="R270"/>
+<instance part="GND34" gate="1" x="203.2" y="96.52" rot="R270"/>
 <instance part="X4" gate="-1" x="10.16" y="121.92" rot="R270"/>
 <instance part="X4" gate="-2" x="-43.18" y="96.52"/>
@@
 <instance part="X8" gate="-1" x="30.48" y="-30.48" rot="R90"/>
 <instance part="X8" gate="-2" x="25.4" y="-30.48" rot="R90"/>
-<instance part="D3" gate="G$1" x="215.9" y="93.98" smashed="yes">
-<attribute name="NAME" x="213.36" y="89.3826" size="1.778" layer="95"/>
-<attribute name="VALUE" x="218.44" y="91.6686" size="1.778" layer="96"/>
-</instance>
 <instance part="P+10" gate="1" x="-10.16" y="76.2" smashed="yes" rot="R90">
 <attribute name="VALUE" x="-10.16" y="76.2" size="1.778" layer="96" rot="R180"/>
@@
 </instance>
 <instance part="GND52" gate="1" x="170.18" y="-10.16"/>
+<instance part="R37" gate="G$1" x="213.36" y="93.98" smashed="yes">
+<attribute name="NAME" x="210.82" y="97.028" size="1.778" layer="95"/>
+<attribute name="VALUE" x="207.518" y="89.662" size="1.778" layer="96"/>
+</instance>
 </instances>
 <busses>
@@
 </segment>
 <segment>
-<wire x1="210.82" y1="96.52" x2="210.82" y2="99.06" width="0.1524" layer="91"/>
-<wire x1="213.36" y1="93.98" x2="210.82" y2="93.98" width="0.1524" layer="91"/>
-<wire x1="210.82" y1="96.52" x2="210.82" y2="93.98" width="0.1524" layer="91"/>
-<junction x="210.82" y="96.52"/>
-<junction x="210.82" y="93.98"/>
+<wire x1="205.74" y1="96.52" x2="205.74" y2="99.06" width="0.1524" layer="91"/>
+<wire x1="205.74" y1="96.52" x2="205.74" y2="93.98" width="0.1524" layer="91"/>
+<junction x="205.74" y="96.52"/>
 <pinref part="X3" gate="-2" pin="KL"/>
 <pinref part="GND34" gate="1" pin="GND"/>
 <pinref part="D4" gate="G$1" pin="A1"/>
-<pinref part="D3" gate="G$1" pin="A"/>
+<pinref part="R37" gate="G$1" pin="2"/>
+<wire x1="205.74" y1="93.98" x2="205.74" y2="91.44" width="0.1524" layer="91"/>
+<wire x1="208.28" y1="93.98" x2="205.74" y2="93.98" width="0.1524" layer="91"/>
+<junction x="205.74" y="93.98"/>
 </segment>
 <segment>
@@
 </segment>
 <segment>
-<wire x1="210.82" y1="109.22" x2="210.82" y2="116.84" width="0.1524" layer="91"/>
-<wire x1="210.82" y1="116.84" x2="220.98" y2="116.84" width="0.1524" layer="91"/>
+<wire x1="205.74" y1="109.22" x2="205.74" y2="116.84" width="0.1524" layer="91"/>
+<wire x1="205.74" y1="116.84" x2="220.98" y2="116.84" width="0.1524" layer="91"/>
 <wire x1="220.98" y1="116.84" x2="220.98" y2="114.3" width="0.1524" layer="91"/>
 <wire x1="220.98" y1="116.84" x2="220.98" y2="119.38" width="0.1524" layer="91"/>
@@
 <net name="N$38" class="0">
 <segment>
+<pinref part="X3" gate="-1" pin="KL"/>
+<pinref part="R13" gate="G$1" pin="1"/>
+<pinref part="R37" gate="G$1" pin="1"/>
+<wire x1="220.98" y1="91.44" x2="220.98" y2="93.98" width="0.1524" layer="91"/>
 <wire x1="218.44" y1="93.98" x2="220.98" y2="93.98" width="0.1524" layer="91"/>
 <junction x="220.98" y="93.98"/>
-<pinref part="X3" gate="-1" pin="KL"/>
-<pinref part="R13" gate="G$1" pin="1"/>
-<pinref part="D3" gate="G$1" pin="C"/>
 </segment>
 </net>
@@
 </segment>
 <segment>
-<wire x1="220.98" y1="104.14" x2="213.36" y2="104.14" width="0.1524" layer="91"/>
+<wire x1="220.98" y1="104.14" x2="208.28" y2="104.14" width="0.1524" layer="91"/>
 <wire x1="220.98" y1="104.14" x2="228.6" y2="104.14" width="0.1524" layer="91"/>
 <junction x="220.98" y="104.14"/>
